Commit message: Configured Mujoco environment in package and added receptacle and april tag in. Works now.

File: src/clr_demos/clr_connector_mating_demo/urdf/receptacle_macro.xacro (robot description, xacro)
@@ -11,9 +11,9 @@
   </joint>
 <!-- ===================== RECEPTACLE ===================== -->
-    <link name="receptacle">
+  <link name="receptacle">
       <visual>
         <origin xyz="0 0 0" rpy="0 0 0"/>
         <geometry>
-          <mesh filename="package://clr_connector_mating_demo/meshes/visual/receptacle.stl"/>
+          <mesh filename="package://clr_connector_mating_demo/meshes/visual/receptacle.stl" scale="0.001 0.001 0.001"/>
         </geometry>
         <material name="receptacle_black">
@@ -24,5 +24,5 @@
         <origin xyz="0 0 0" rpy="0 0 0"/>
         <geometry>
-          <mesh filename="package://clr_connector_mating_demo/meshes/visual/receptacle.stl"/>
+          <mesh filename="package://clr_connector_mating_demo/meshes/visual/receptacle.stl" scale="0.001 0.001 0.001"/>
         </geometry>
       </collision>
@@ -42,5 +42,5 @@
      <parent link="receptacle"/>
      <child link="apriltag_0"/>
-     <origin xyz="0 0 0" rpy="0 0 0"/>
+     <origin xyz="0 -0.105 0.0127" rpy="0 1.57 1.57"/>
    </joint>
   </xacro:macro>
